File: Level_Shift.kicad_sch (KiCad schematic)
At the start: 7 parts, among them U24 74AVC4T245, U29 74LVC8T245

Commit message: Added Level Shifter schematic & moved symbols
- Created a separate Level Shifter schematic to prepare use of some gates for Digital output enables.
Parts:
- removed C135, C137, C63, C64: 100nF, Capacitor_SMD:C_0402_1005Metric, symbol Device:C_Small
- removed R69: 4.75k, Resistor_SMD:R_0402_1005Metric, symbol Device:R_Small_US
- removed U24: 74AVC4T245, Package_SO:TSSOP-16_4.4x5mm_P0.65mm, symbol evr-fmc:74LVC4T245
- removed U29: 74LVC8T245, Package_SO:TSSOP-24_4.4x7.8mm_P0.65mm, symbol evr-fmc:74LVC8T245
- added C65, C66, C67, C68, C69, C70, C71, C72: 100nF, Capacitor_SMD:C_0402_1005Metric, symbol Device:C_Small
- added R68, R70, R89, R90, R91, R92, R93, R94, R96, R97: 4.75k, Resistor_SMD:R_0402_1005Metric, symbol Device:R_Small_US
- added U23, U25: 74AVC4T245, Package_SO:TSSOP-16_4.4x5mm_P0.65mm, symbol evr-fmc:74LVC4T245
- added U26, U27: 74LVC8T245, Package_SO:TSSOP-24_4.4x7.8mm_P0.65mm, symbol evr-fmc:74LVC8T245
Connections:
- net GND: now also C65.1, C66.1, C67.1, C68.1, C69.1, C70.1, C71.1, C72.1, R93.1, R94.1, U23.2 (1DIR), U23.3 (2DIR), U23.8 (GND), U23.9 (GND), U25.2 (1DIR), U25.3 (2DIR), U25.8 (GND), U25.9 (GND), U26.11 (GND), U26.12 (GND), U26.13 (GND), U26.22 (OE), U27.11 (GND), U27.12 (GND), U27.13 (GND), U27.22 (OE)
- net VDD3P3V: now also C65.2, C67.2, C70.2, C72.2, U23.16 (VCCB), U25.16 (VCCB), U26.23 (VCCB), U26.24 (VCCB), U27.23 (VCCB), U27.24 (VCCB)
- new net: R68.1, U26.2 (DIR)
- new net: R70.1, U27.2 (DIR)
- new net Cleaner_0.INTR: U23.13 (B1)
- new net Cleaner_0.LOL: U23.11 (B3)
- new net Cleaner_0.LOS_XO: U23.12 (B2)
- new net Cleaner_0.OE: U26.21 (B1)
- new net Cleaner_0.RST: U26.16 (B6)
- new net Cleaner_0.SPI_CLK: U26.19 (B3)
- new net Cleaner_0.SPI_CS: U26.17 (B5)
- new net Cleaner_0.SPI_SDI: U26.20 (B2)
- new net Cleaner_0.SPI_SDO: U23.10 (B4)
- new net Cleaner_1.INTR: U25.13 (B1)
- new net Cleaner_1.LOL: U25.11 (B3)
- new net Cleaner_1.LOS_XO: U25.12 (B2)
- new net Cleaner_1.OE: U27.21 (B1)
- new net Cleaner_1.RST: U27.16 (B6)
- new net Cleaner_1.SPI_CLK: U27.19 (B3)
- new net Cleaner_1.SPI_CS: U27.17 (B5)
- new net Cleaner_1.SPI_SDI: U27.20 (B2)
- new net Cleaner_1.SPI_SDO: U25.10 (B4)
- new net Cleaner_SPI_0.CLK: U26.5 (A3)
- new net Cleaner_SPI_0.CS: R89.1, U26.7 (A5)
- new net Cleaner_SPI_0.OE: R91.1, U26.3 (A1)
- new net Cleaner_SPI_0.SDI: U26.4 (A2)
- new net Cleaner_SPI_0.SDO: U23.7 (A4)
- new net Cleaner_SPI_1.CLK: U27.5 (A3)
- new net Cleaner_SPI_1.CS: R90.1, U27.7 (A5)
- new net Cleaner_SPI_1.OE: R92.1, U27.3 (A1)
- new net Cleaner_SPI_1.SDI: U27.4 (A2)
- new net Cleaner_SPI_1.SDO: U25.7 (A4)
- new net Fault_0.INTR: U23.4 (A1)
- new net Fault_0.LOL: U23.6 (A3)
- new net Fault_0.LOS_XO: U23.5 (A2)
- new net Fault_1.INTR: U25.4 (A1)
- new net Fault_1.LOL: U25.6 (A3)
- new net Fault_1.LOS_XO: U25.5 (A2)
- new net OE_Faults_0: R96.1, U23.14 (OE), U23.15 (OE)
- new net OE_Faults_1: R97.1, U25.14 (OE), U25.15 (OE)
- new net VADJ: C66.2, C68.2, C69.2, C71.2, R68.2, R70.2, R89.2, R90.2, R91.2, R92.2, R96.2, R97.2, U23.1 (VCCA), U25.1 (VCCA), U26.1 (VCCA), U27.1 (VCCA)
- new net ~{RST}_0: R93.2, U26.8 (A6)
- new net ~{RST}_1: R94.2, U27.8 (A6)
- no-connect marks 1 -> 12
Other:
- note added: "Held in ~{RST} until power up"
