File: eeprom.kicad_sch (KiCad schematic)
At the start: 9 parts, among them J19 WP Jumper, U9 AT24C64D

Commit message: Final Draft - Ready to Review
Things to do:
Round diff traces before generting fabrication files
Change name of project to 'trigger output fmc'
Align this with recent updates to fmc-template

Updates:
- Cleaned up BOM
- Arranged silkscreen and fab layers
- Shortened power traces from LDOs to Jitter Cleaner IC
- Fixed traces/planes with sharp corners
- Straightened out all MMCX Test Ports
Parts:
- C33: MPN GCM188R71E105KA64D -> GCM188R71C105KA64D; Manufacturer Murata Electronics -> Murata
Changed lines of the file:
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@@
 			)
 		)
-		(property "MPN" "GCM188R71E105KA64D"
+		(property "MPN" "GCM188R71C105KA64D"
 			(at 133.35 86.36 0)
 			(effects
@@
 			)
 		)
-		(property "Manufacturer" "Murata Electronics"
+		(property "Manufacturer" "Murata"
 			(at 133.35 86.36 0)
 			(effects

Commit message: Final Draft - Ready for review
Updates:
- Changed area behind FMC connector to match the new Osprey FMC template
  - This includes a new 12V LED, more robust power input traces, arranged elements for readability.

Things to do:
Round diff traces before generating fabrication files
Change name of project to 'trigger output fmc'
Connections:
- net P1_3P3VAUX renamed 3P3VAUX
Other:
- title: FMC Template -> Trigger Output FMC
Changed lines of the file:
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@@
 	(paper "USLetter")
 	(title_block
-		(title "FMC Template")
-		(date "2026-01-26")
+		(title "Trigger Output FMC")
+		(date "2026-05-07")
 		(rev "1.0")
 		(company "SPDX-FileCopyrightText: 2025 Osprey DCS")
@@
 		)
 	)
-	(global_label "P1_3P3VAUX"
+	(global_label "3P3VAUX"
 		(shape input)
 		(at 130.81 81.28 180)
@@
 		)
 		(property "Intersheetrefs" "${INTERSHEET_REFS}"
-			(at 116.0509 81.28 0)
+			(at 119.4186 81.28 0)
 			(effects
 				(font
@@
 		)
 	)
-	(global_label "P1_3P3VAUX"
+	(global_label "3P3VAUX"
 		(shape input)
 		(at 101.6 104.14 180)
@@
 		)
 		(property "Intersheetrefs" "${INTERSHEET_REFS}"
-			(at 86.7615 104.14 0)
+			(at 90.2086 104.14 0)
 			(effects
 				(font
