File: eeprom.kicad_sch (KiCad schematic)
At the start: 9 parts, among them J19 WP Jumper, U9 AT24C64D

Commit message: Fixed Silkscreen and BOM
All DRC/ERC errors are resolved.
Parts:
- C33: Digikey (none) -> 490-5241-6-ND
- J19: Digikey (none) -> 952-2261-ND
- R10, R11, R12, R14, R15: Digikey (none) -> 13-RC0603FR-134K75LDKR-ND
- R13: Digikey (none) -> 311-11.5KHRDKR-ND
- U9: Digikey (none) -> AT24C64D-SSHM-TDKR-ND
Changed lines of the file:
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@@
+			)
+		)
+		(property "Digikey" "13-RC0603FR-134K75LDKR-ND"
+			(at 105.41 99.06 90)
+			(effects
+				(font
+					(size 1.27 1.27)
+				)
+				(hide yes)
 			)
 		)
@@
 			)
 		)
+		(property "Digikey" "311-11.5KHRDKR-ND"
+			(at 151.13 90.17 0)
+			(effects
+				(font
+					(size 1.27 1.27)
+				)
+				(hide yes)
+			)
+		)
 		(pin "1"
 		)
@@
 			)
 		)
+		(property "Digikey" "AT24C64D-SSHM-TDKR-ND"
+			(at 138.43 101.6 0)
+			(effects
+				(font
+					(size 1.27 1.27)
+				)
+				(hide yes)
+			)
+		)
 		(pin "1"
 		)
@@
 			)
 		)
-		(property "Description" "CAP CER 1UF 25V X7R 0603"
+		(property "Description" "CAP CER 1UF 16V X7R 0603"
 			(at 133.35 86.36 0)
 			(effects
@@
 			)
 		)
+		(property "Digikey" "490-5241-6-ND"
+			(at 133.35 86.36 0)
+			(effects
+				(font
+					(size 1.27 1.27)
+				)
+				(hide yes)
+			)
+		)
 		(pin "1"
 		)
@@
 			)
 		)
+		(property "Digikey" "13-RC0603FR-134K75LDKR-ND"
+			(at 167.64 93.98 0)
+			(effects
+				(font
+					(size 1.27 1.27)
+				)
+				(hide yes)
+			)
+		)
 		(pin "1"
 		)
@@
 			)
 		)
+		(property "Digikey" "13-RC0603FR-134K75LDKR-ND"
+			(at 121.92 104.14 90)
+			(effects
+				(font
+					(size 1.27 1.27)
+				)
+				(hide yes)
+			)
+		)
 		(pin "1"
 		)
@@
 			)
 		)
+		(property "Digikey" "13-RC0603FR-134K75LDKR-ND"
+			(at 115.57 101.6 90)
+			(effects
+				(font
+					(size 1.27 1.27)
+				)
+				(hide yes)
+			)
+		)
 		(pin "1"
 		)
@@
 			)
 		)
+		(property "Digikey" "952-2261-ND"
+			(at 161.29 107.95 0)
+			(effects
+				(font
+					(size 1.27 1.27)
+				)
+				(hide yes)
+			)
+		)
 		(pin "1"
 		)
@@
 			(at 175.26 93.98 0)
 			(effects
+				(font
+					(size 1.27 1.27)
+				)
+				(hide yes)
+			)
+		)
+		(property "Digikey" "13-RC0603FR-134K75LDKR-ND"
+			(at 175.26 93.98 0)
+			(effects

Commit message: Final Draft for project
- Changed LDO for Digital Output driver to a LP3855-ADJ
- Aligned Digital Output driver sections
- Added Additional Capacitance on each digital output drive channel
- Revised Differential Lines geometry on top layer
- Revised Power routing and internal planes
Parts:
- C33: Digikey 490-5241-6-ND -> (none)
- J19: Digikey 952-2261-ND -> (none)
- R10, R11, R12, R14, R15: Digikey 13-RC0603FR-134K75LDKR-ND -> (none)
- R13: Digikey 311-11.5KHRDKR-ND -> (none)
- U9: Digikey AT24C64D-SSHM-TDKR-ND -> (none)
Changed lines of the file:
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@@
-			)
-		)
-		(property "Digikey" "13-RC0603FR-134K75LDKR-ND"
-			(at 105.41 99.06 90)
-			(effects
-				(font
-					(size 1.27 1.27)
-				)
-				(hide yes)
 			)
 		)
@@
 			)
 		)
-		(property "Digikey" "311-11.5KHRDKR-ND"
-			(at 151.13 90.17 0)
-			(effects
-				(font
-					(size 1.27 1.27)
-				)
-				(hide yes)
-			)
-		)
 		(pin "1"
 		)
@@
 			)
 		)
-		(property "Digikey" "AT24C64D-SSHM-TDKR-ND"
-			(at 138.43 101.6 0)
-			(effects
-				(font
-					(size 1.27 1.27)
-				)
-				(hide yes)
-			)
-		)
 		(pin "1"
 		)
@@
 			)
 		)
-		(property "Digikey" "490-5241-6-ND"
-			(at 133.35 86.36 0)
-			(effects
-				(font
-					(size 1.27 1.27)
-				)
-				(hide yes)
-			)
-		)
 		(pin "1"
 		)
@@
 			)
 		)
-		(property "Digikey" "13-RC0603FR-134K75LDKR-ND"
-			(at 167.64 93.98 0)
-			(effects
-				(font
-					(size 1.27 1.27)
-				)
-				(hide yes)
-			)
-		)
 		(pin "1"
 		)
@@
 			)
 		)
-		(property "Digikey" "13-RC0603FR-134K75LDKR-ND"
-			(at 121.92 104.14 90)
-			(effects
-				(font
-					(size 1.27 1.27)
-				)
-				(hide yes)
-			)
-		)
 		(pin "1"
 		)
@@
 			)
 		)
-		(property "Digikey" "13-RC0603FR-134K75LDKR-ND"
-			(at 115.57 101.6 90)
-			(effects
-				(font
-					(size 1.27 1.27)
-				)
-				(hide yes)
-			)
-		)
 		(pin "1"
 		)
@@
 			)
 		)
-		(property "Digikey" "952-2261-ND"
-			(at 161.29 107.95 0)
-			(effects
-				(font
-					(size 1.27 1.27)
-				)
-				(hide yes)
-			)
-		)
 		(pin "1"
 		)
@@
 			(at 175.26 93.98 0)
 			(effects
-				(font
-					(size 1.27 1.27)
-				)
-				(hide yes)
-			)
-		)
-		(property "Digikey" "13-RC0603FR-134K75LDKR-ND"
-			(at 175.26 93.98 0)
-			(effects
