File: fmc.kicad_sch (KiCad schematic)
At the start: 31 parts, among them P1 ASP-134488-01, Q1 FDN335N, Q2 FDN335N, Q3 FDN335N

Commit message: Routed LVDS lines
- Routed LVDS lines
- Swapped some digital output pairs
- Properly connected the output enable signal for digital outputs in the schematic
Connections:
- net D_Output10.N: now also P1.G31; no longer P1.G22
- net D_Output10.P: now also P1.G30; no longer P1.G21
- net D_Output11.N: now also P1.H32; no longer P1.G28
- net D_Output11.P: now also P1.H31; no longer P1.G27
- net D_Output12.N: now also P1.G34; no longer P1.G31
- net D_Output12.P: now also P1.G33; no longer P1.G30
- net D_Output13.N: now also P1.H35; no longer P1.H32
- net D_Output13.P: now also P1.H34; no longer P1.H31
- net D_Output14.N: now also P1.H38; no longer P1.G34
- net D_Output14.P: now also P1.H37; no longer P1.G33
- net D_Output15.N: now also P1.G37; no longer P1.H35
- net D_Output15.P: now also P1.G36; no longer P1.H34
- net D_Output2.N: now also P1.G16; no longer P1.D15
- net D_Output2.P: now also P1.G15; no longer P1.D14
- net D_Output3.N: now also P1.D15; no longer P1.C15
- net D_Output3.P: now also P1.D14; no longer P1.C14
- net D_Output4.N: now also P1.C15; no longer P1.G16
- net D_Output4.P: now also P1.C14; no longer P1.G15
- net D_Output5.N: now also P1.G19; no longer P1.H17
- net D_Output5.P: now also P1.G18; no longer P1.H16
- net D_Output8.N: now also P1.G22; no longer P1.G19
- net D_Output8.P: now also P1.G21; no longer P1.G18
- net D_Output9.N: now also P1.G28; no longer P1.H20
- net D_Output9.P: now also P1.G27; no longer P1.H19
- net OE_Digital_Outputs: now also P1.H19; no longer P1.G36
Changed lines of the file:
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@@
 	)
 	(no_connect
-		(at 314.96 118.11)
-	)
-	(no_connect
 		(at 125.73 208.28)
 	)
@@
 	)
 	(no_connect
+		(at 379.73 64.77)
+	)
+	(no_connect
 		(at 180.34 172.72)
 	)
@@
 	)
 	(no_connect
-		(at 381 118.11)
-	)
-	(no_connect
 		(at 125.73 185.42)
 	)
@@
 	)
 	(no_connect
+		(at 379.73 67.31)
+	)
+	(no_connect
 		(at 256.54 194.31)
 	)
@@
 	)
 	(no_connect
+		(at 379.73 74.93)
+	)
+	(no_connect
 		(at 284.48 224.79)
 	)
@@
 	)
 	(no_connect
-		(at 381 120.65)
-	)
-	(no_connect
 		(at 204.47 231.14)
 	)
@@
 		)
 	)
+	(wire
+		(pts
+			(xy 360.68 118.11) (xy 403.86 118.11)
+		)
+		(stroke
+			(width 0)
+			(type default)
+		)
+	)
 	(bus
 		(pts
@@
 	(wire
 		(pts
+			(xy 379.73 64.77) (xy 403.86 64.77)
+		)
+		(stroke
+			(width 0)
+			(type default)
+		)
+	)
+	(wire
+		(pts
 			(xy 252.73 242.57) (xy 256.54 242.57)
 		)
@@
 	(wire
 		(pts
-			(xy 360.68 67.31) (xy 403.86 67.31)
-		)
-		(stroke
-			(width 0)
-			(type default)
-		)
-	)
-	(wire
-		(pts
 			(xy 123.19 210.82) (xy 125.73 210.82)
 		)
@@
 	(wire
 		(pts
-			(xy 360.68 72.39) (xy 403.86 72.39)
+			(xy 300.99 115.57) (xy 339.09 115.57)
 		)
 		(stroke
@@
 	(wire
 		(pts
-			(xy 123.19 213.36) (xy 123.19 220.98)
+			(xy 379.73 67.31) (xy 403.86 67.31)
 		)
 		(stroke
@@
 	(wire
 		(pts
-			(xy 300.99 95.25) (xy 339.09 95.25)
+			(xy 123.19 213.36) (xy 123.19 220.98)
 		)
 		(stroke
@@
 	(wire
 		(pts
-			(xy 300.99 110.49) (xy 339.09 110.49)
+			(xy 300.99 95.25) (xy 339.09 95.25)
 		)
 		(stroke
@@
 	(wire
 		(pts
-			(xy 336.55 125.73) (xy 339.09 125.73)
+			(xy 300.99 110.49) (xy 339.09 110.49)
 		)
 		(stroke
@@
 	(wire
 		(pts
-			(xy 177.8 165.1) (xy 180.34 165.1)
+			(xy 336.55 125.73) (xy 339.09 125.73)
 		)
 		(stroke
@@
 	(wire
 		(pts
-			(xy 280.67 143.51) (xy 280.67 146.05)
+			(xy 177.8 165.1) (xy 180.34 165.1)
 		)
 		(stroke
@@
 	(wire
 		(pts
-			(xy 401.32 77.47) (xy 401.32 69.85)
+			(xy 280.67 143.51) (xy 280.67 146.05)
 		)
 		(stroke
@@
 	(wire
 		(pts
-			(xy 381 118.11) (xy 403.86 118.11)
+			(xy 401.32 77.47) (xy 401.32 69.85)
 		)
 		(stroke
@@
 	(wire
 		(pts
-			(xy 360.68 64.77) (xy 403.86 64.77)
-		)
-		(stroke
-			(width 0)
-			(type default)
-		)
-	)
-	(wire
-		(pts
 			(xy 379.73 82.55) (xy 403.86 82.55)
 		)
@@
 	(wire
 		(pts
+			(xy 360.68 120.65) (xy 403.86 120.65)
+		)
+		(stroke
+			(width 0)
+			(type default)
+		)
+	)
+	(wire
+		(pts
 			(xy 300.99 87.63) (xy 339.09 87.63)
 		)
@@
 	(wire
 		(pts
+			(xy 360.68 72.39) (xy 403.86 72.39)
+		)
+		(stroke
+			(width 0)
+			(type default)
+		)
+	)
+	(wire
+		(pts
 			(xy 349.25 184.15) (xy 349.25 186.69)
 		)
@@
 	(wire
 		(pts
-			(xy 314.96 118.11) (xy 339.09 118.11)
-		)
-		(stroke
-			(width 0)
-			(type default)
-		)
-	)
-	(wire
-		(pts
 			(xy 200.66 182.88) (xy 200.66 190.5)
 		)
@@
 	(wire
 		(pts
-			(xy 360.68 74.93) (xy 403.86 74.93)
+			(xy 300.99 118.11) (xy 339.09 118.11)
 		)
 		(stroke
@@
 	(wire
 		(pts
+			(xy 379.73 74.93) (xy 403.86 74.93)
+		)
+		(stroke
+			(width 0)
+			(type default)
+		)
+	)
+	(wire
+		(pts
 			(xy 224.79 162.56) (xy 224.79 170.18)
 		)
@@
 	(wire
 		(pts
-			(xy 381 120.65) (xy 403.86 120.65)
-		)
-		(stroke
-			(width 0)
-			(type default)
-		)
-	)
-	(wire
-		(pts
 			(xy 227.33 43.18) (xy 274.32 43.18)
 		)
@@
 	(wire
 		(pts
-			(xy 300.99 115.57) (xy 339.09 115.57)
-		)
-		(stroke
-			(width 0)
-			(type default)
-		)
-	)
-	(wire
-		(pts
 			(xy 284.48 153.67) (xy 280.67 153.67)
 		)
@@
 		)
 	)
-	(label "D_Output13.N"
+	(label "D_Output11.N"
 		(at 360.68 105.41 0)
 		(effects
@@
 		)
 	)
-	(label "D_Output2.N"
+	(label "D_Output3.N"
 		(at 227.33 60.96 0)
 		(effects
@@
 		)
 	)
-	(label "D_Output12.P"
+	(label "D_Output10.P"
 		(at 300.99 100.33 0)
 		(effects
@@
 		)
 	)
-	(label "D_Output12.N"
+	(label "D_Output10.N"
 		(at 300.99 102.87 0)
 		(effects
@@
 		)
 	)
-	(label "D_Output14.P"
+	(label "D_Output12.P"
 		(at 300.99 107.95 0)
 		(effects
@@
 		)
 	)
-	(label "D_Output5.P"
-		(at 360.68 64.77 0)
-		(effects
-			(font
-				(size 1.27 1.27)
-			)
-			(justify left bottom)
-		)
-	)
 	(label "OE_Digital_Outputs"
-		(at 300.99 115.57 0)
+		(at 360.68 72.39 0)
 		(effects
 			(font
@@
 		)
 	)
-	(label "D_Output4.N"
+	(label "D_Output2.N"
 		(at 300.99 64.77 0)
 		(effects
@@
 		)
 	)
-	(label "D_Output8.P"
+	(label "D_Output5.P"
 		(at 300.99 69.85 0)
 		(effects
@@
 		)
 	)
-	(label "D_Output4.P"
+	(label "D_Output14.P"
+		(at 360.68 118.11 0)
+		(effects
+			(font
+				(size 1.27 1.27)
+			)
+			(justify left bottom)
+		)
+	)
+	(label "D_Output2.P"
 		(at 300.99 62.23 0)
 		(effects
@@
 		)
 	)
-	(label "D_Output3.P"
+	(label "D_Output4.P"
 		(at 156.21 58.42 0)
 		(effects
@@
 		)
 	)
-	(label "D_Output11.P"
+	(label "D_Output9.P"
 		(at 300.99 92.71 0)
 		(effects
@@
 		)
 	)
-	(label "D_Output10.P"
+	(label "D_Output8.P"
 		(at 300.99 77.47 0)
 		(effects
@@
 		)
 	)
+	(label "D_Output14.N"
+		(at 360.68 120.65 0)
+		(effects
+			(font
+				(size 1.27 1.27)
+			)
+			(justify left bottom)
+		)
+	)
 	(label "OE_Digital_Outputs"
 		(at 140.97 15.24 180)
@@
 		)
 	)
-	(label "D_Output10.N"
+	(label "D_Output8.N"
 		(at 300.99 80.01 0)
 		(effects
@@
 		)
 	)
-	(label "D_Output15.N"
+	(label "D_Output13.N"
 		(at 360.68 113.03 0)
 		(effects
@@
 		)
 	)
-	(label "D_Output2.P"
+	(label "D_Output3.P"
 		(at 227.33 58.42 0)
 		(effects
@@
 		)
 	)
-	(label "D_Output13.P"
+	(label "D_Output11.P"
 		(at 360.68 102.87 0)
 		(effects
@@
 		)
 	)
-	(label "D_Output9.N"
-		(at 360.68 74.93 0)
+	(label "D_Output15.N"
+		(at 300.99 118.11 0)
 		(effects
 			(font
@@
 		)
 	)
-	(label "D_Output8.N"
+	(label "D_Output5.N"
 		(at 300.99 72.39 0)
 		(effects
@@
 		)
 	)
-	(label "D_Output5.N"
-		(at 360.68 67.31 0)
-		(effects
-			(font
-				(size 1.27 1.27)
-			)
-			(justify left bottom)
-		)
-	)
 	(label "Cleaner_~{RST}_1"
 		(at 86.36 111.76 180)
@@
 		)
 	)
-	(label "D_Output15.P"
+	(label "D_Output13.P"
 		(at 360.68 110.49 0)
 		(effects
@@
 		)
 	)
-	(label "D_Output3.N"
+	(label "D_Output4.N"
 		(at 156.21 60.96 0)
 		(effects
@@
 		)
 	)
-	(label "D_Output11.N"
+	(label "D_Output9.N"
 		(at 300.99 95.25 0)
 		(effects
@@
 		)
 	)
-	(label "D_Output14.N"
+	(label "D_Output12.N"
 		(at 300.99 110.49 0)
 		(effects
@@
 		)
 	)
-	(label "D_Output9.P"
-		(at 360.68 72.39 0)
+	(label "D_Output15.P"
+		(at 300.99 115.57 0)
 		(effects
 			(font

Commit message: Fixed Silkscreen and BOM
All DRC/ERC errors are resolved.
Parts:
- C34, C35, C79: Digikey (none) -> 1276-6780-6-ND; MPN GRM21BR61E226ME44L -> CL21A226MOCLRNC; Manufacturer Murata -> Samsung
- D1, D2, D3, D4, D5: Digikey (none) -> 754-1116-6-ND
- P1: Digikey (none) -> SAM8730-ND
- Q1, Q2, Q3: Digikey (none) -> FDN335NDKR-ND
- R100: Digikey (none) -> 311-8.20KHRDKR-ND
- R101, R102, R103: Digikey (none) -> 311-100KHRDKR-ND
- R16, R17: Digikey (none) -> P0.0GDKR-ND
- R18, R19, R20, R95: Digikey (none) -> RHM1.00KADDKR-ND
- TP1: Digikey (none) -> 36-5001-ND
- TP2, TP3, TP4: Digikey (none) -> 36-5000-ND

Commit message: Changed mechanical holes to universal Mable footprints
Parts:
- H1: footprint MountingHole:MountingHole_2.7mm_M2.5_Pad -> rf-input-fmc:MountingHole_3.0mm_M2.5_Pad_3.3mm_UniversalMarbleSlot
- H3, H4: footprint rf-input-fmc:MountingHole_2.7mm_Pad_3.1mm -> rf-input-fmc:MountingHole_3.0mm_3.8mm_Pad_3.3mm_UniversalMarbleSlot
Changed lines of the file:
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@@
 			)
 		)
-		(property "Footprint" "rf-input-fmc:MountingHole_2.7mm_Pad_3.1mm"
+		(property "Footprint" "rf-input-fmc:MountingHole_3.0mm_3.8mm_Pad_3.3mm_UniversalMarbleSlot"
 			(at 59.69 226.06 0)
 			(effects
@@
 			)
 		)
-		(property "Footprint" "rf-input-fmc:MountingHole_2.7mm_Pad_3.1mm"
+		(property "Footprint" "rf-input-fmc:MountingHole_3.0mm_3.8mm_Pad_3.3mm_UniversalMarbleSlot"
 			(at 59.69 237.49 0)
 			(effects
@@
 			)
 		)
-		(property "Footprint" "MountingHole:MountingHole_2.7mm_M2.5_Pad"
+		(property "Footprint" "rf-input-fmc:MountingHole_3.0mm_M2.5_Pad_3.3mm_UniversalMarbleSlot"
 			(at 59.69 203.2 0)
 			(effects

Commit message: Final Draft for project
- Changed LDO for Digital Output driver to a LP3855-ADJ
- Aligned Digital Output driver sections
- Added Additional Capacitance on each digital output drive channel
- Revised Differential Lines geometry on top layer
- Revised Power routing and internal planes
Parts:
- C34, C35, C79: Digikey 1276-6780-6-ND -> (none)
- D1, D2, D3, D4, D5: Digikey 754-1116-6-ND -> (none)
- P1: Digikey SAM8730-ND -> (none)
- Q1, Q2, Q3: Digikey FDN335NDKR-ND -> (none)
- R100: Digikey 311-8.20KHRDKR-ND -> (none)
- R101, R102, R103: Digikey 311-100KHRDKR-ND -> (none)
- R16, R17: Digikey P0.0GDKR-ND -> (none)
- R18, R19, R20, R95: Digikey RHM1.00KADDKR-ND -> (none)
- TP1: Digikey 36-5001-ND -> (none)
- TP2, TP3, TP4: Digikey 36-5000-ND -> (none)

Commit message: Schematic and Layout Tweaks
- Updated all vias to 0.6/0.3mm
- New mechanical universal Marble holes for H2
- widen the power traces to Test points
- Add pin 4 of U20/U24 to GND net
- add a GND pour around U44 for heat
- Widen GND traces on LDOs (U24/U20)
- Grounding of unused gates of level shifters
-Small updates footprints for U18,U19,U23,U25
Parts:
- H2: footprint rf-input-fmc:MountingHole_2.7mm_M2.5_Pad_Marble_Slot -> rf-input-fmc:MountingHole_3.0mm_M2.5_Pad_3.3mm_UniversalMarbleSlot
Changed lines of the file:
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@@
 			)
 		)
-		(property "Footprint" "rf-input-fmc:MountingHole_2.7mm_M2.5_Pad_Marble_Slot"
+		(property "Footprint" "rf-input-fmc:MountingHole_3.0mm_M2.5_Pad_3.3mm_UniversalMarbleSlot"
 			(at 59.69 214.63 0)
 			(effects
