File: trigger-output-fmc.kicad_pcb (KiCad board)
At the start: 8 copper layers, 84 x 69 mm, 340 parts, among them J1 MMCX, J10 MMCX, J11 MMCX, J12 MMCX, J13 MMCX, J14 MMCX, J15 MMCX, J16 MMCX, J19 WP Jumper, J2 MMCX, J3 MMCX, J4 MMCX, J5 MMCX, J6 MMCX, J7 MMCX, J8 MMCX, J9 MMCX, P1 ASP-134488-01, Q1 FDN335N, Q2 FDN335N, Q3 FDN335N, T1 TCM2-43X+, T2 TCM2-43X+, T3 TCM2-43X+, T4 TCM2-43X+, U1 TLV3601, U10 SN74LVC2G126, U11 TLV3601, U12 SN74LVC2G126, U13 TLV3601, U14 SN74LVC2G126, U15 TLV3601, U16 SN74LVC2G126, U17 TLV3601, U18 SI5394, U19 SI5394, U2 TLV3601, U20 TLV75733PDBV, U21 TLV75718PDBV, U22 TPS563200, U23 74AVC4T245, U24 TLV75733PDBV, U25 74AVC4T245, U26 74LVC8T245, U27 74LVC8T245, U28 TLV75718PDBV, U29 SN74LVC2G126, U3 TLV3601, U30 TLV3601, U31 SN74LVC2G126, U32 TLV3601, U33 SN74LVC2G126, U34 TLV3601, U35 SN74LVC2G126, U36 TLV3601, U37 SN74LVC2G126, U38 TLV3601, U39 SN74LVC2G126, U4 SN74LVC2G126, U40 TLV3601, U41 SN74LVC2G126, U42 TLV3601, U43 SN74LVC2G126, U44 LP3855EMP-ADJ/NOPB, U48 SN74LVC2G126, U5 SN74LVC2G126, U6 TLV3601, U7 SN74LVC2G126, U8 TLV3601, U9 AT24C64D, Y1 CX3225SB48000D0FPJC1, Y2 CX3225SB48000D0FPJC1

Commit message: Updated Version Number to 1.1
Updated Version Number to 1.1
-Added Test point for digital output LDO supply (TP10)
Parts:
- added TP10: Keystone5000, TestPoint:TestPoint_Keystone_5000-5004_Miniature, F.Cu at (137.0, 76.8)
Other:
- board text added: "5.0V"
- board text added: "Trigger Output FMC 1.1 Osprey DCS 2026"
- board text removed: "Trigger Output FMC 1.0 Osprey DCS 2026"
Changed lines of the file:
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@@
 	(title_block
 		(title "Trigger Output FMC")
-		(date "2026-05-07")
-		(rev "1.0")
+		(date "2026-10-06")
+		(rev "1.1")
 		(company "SPDX-FileCopyrightText: 2025 Osprey DCS")
 		(comment 1 "SPDX-License-Identifier: CERN-OHL-S-2.0+")
@@
 		)
 	)
+	(footprint "TestPoint:TestPoint_Keystone_5000-5004_Miniature"
+		(layer "F.Cu")
+		(at 137 76.75)
+		(descr "Keystone THM Miniature Test Point 5000-5004, http://www.keyelco.com/product-pdf.cfm?p=1309")
+		(tags "Through Hole Mount Test Points")
+		(property "Reference" "TP10"
+			(at 0 -2.5 0)
+			(layer "F.SilkS")
+			(hide yes)
+			(effects
+				(font
+					(size 1 1)
+					(thickness 0.15)
+				)
+			)
+		)
+		(property "Value" "Keystone5000"
+			(at 0 2.5 0)
+			(layer "F.Fab")
+			(hide yes)
+			(effects
+				(font
+					(size 1 1)
+					(thickness 0.15)
+				)
+			)
+		)
+		(property "Datasheet" "~"
+			(at 0 0 0)
+			(unlocked yes)
+			(layer "F.Fab")
+			(hide yes)
+			(effects
+				(font
+					(size 1.27 1.27)
+					(thickness 0.15)
+				)
+			)
+		)
+		(property "Description" "PC TEST POINT MINIATURE RED"
+			(at 0 0 0)
+			(unlocked yes)
+			(layer "F.Fab")
+			(hide yes)
+			(effects
+				(font
+					(size 1.27 1.27)
+					(thickness 0.15)
+				)
+			)
+		)
+		(property "MPN" "5000"
+			(at 0 0 0)
+			(unlocked yes)
+			(layer "F.Fab")
+			(hide yes)
+			(effects
+				(font
+					(size 1 1)
+					(thickness 0.15)
+				)
+			)
+		)
+		(property "Manufacturer" "Keystone Electronics"
+			(at 0 0 0)
+			(unlocked yes)
+			(layer "F.Fab")
+			(hide yes)
+			(effects
+				(font
+					(size 1 1)
+					(thickness 0.15)
+				)
+			)
+		)
+		(property ki_fp_filters "Pin* Test*")
+		(sheetname "/Digital IO/")
+		(sheetfile "Digital_IO.kicad_sch")
+		(attr through_hole dnp)
+		(fp_circle
+			(center 0 0)
+			(end 1.4 0)
+			(stroke
+				(width 0.12)
+				(type solid)
+			)
+			(fill no)
+			(layer "F.SilkS")
+		)
+		(fp_circle
+			(center 0 0)
+			(end 1.65 0)
+			(stroke
+				(width 0.05)
+				(type solid)
+			)
+			(fill no)
+			(layer "F.CrtYd")
+		)
+		(fp_rect
+			(start -0.75 -0.25)
+			(end 0.75 0.25)
+			(stroke
+				(width 0.1)
+				(type default)
+			)
+			(fill no)
+			(layer "F.Fab")
+		)
+		(fp_circle
+			(center 0 0)
+			(end 1.25 0)
+			(stroke
+				(width 0.1)
+				(type solid)
+			)
+			(fill no)
+			(layer "F.Fab")
+		)
+		(fp_text user "${REFERENCE}"
+			(at 0 -2.5 0)
+			(layer "F.Fab")
+			(effects
+				(font
+					(size 1 1)
+					(thickness 0.15)
+				)
+			)
+		)
+		(pad "1" thru_hole circle
+			(at 0 0)
+			(size 2 2)
+			(drill 1)
+			(layers "*.Cu" "*.Mask")
+			(remove_unused_layers no)
+			(net 53 "/Digital IO/VCC")
+			(pinfunction "1")
+			(pintype "passive")
+		)
+		(embedded_fonts no)
+		(model "${KICAD9_3DMODEL_DIR}/TestPoint.3dshapes/TestPoint_Keystone_5000-5004_Miniature.step"
+			(offset
+				(xyz 0 0 0)
+			)
+			(scale
+				(xyz 1 1 1)
+			)
+			(rotate
+				(xyz 0 0 0)
+			)
+		)
+	)
 	(footprint "Capacitor_SMD:C_0805_2012Metric"
 		(layer "F.Cu")
@@
 		)
 	)
-	(gr_text "Trigger Output FMC 1.0\nOsprey DCS 2026\n"
+	(gr_text "Trigger Output FMC 1.1\nOsprey DCS 2026\n"
 		(at 186.03 89.625 90)
 		(layer "F.SilkS")
@@
 		)
 	)
+	(gr_text "5.0V\n"
+		(at 137 74.5 0)
+		(layer "F.SilkS")
+		(effects
+			(font
+				(size 1 1)
+				(thickness 0.15)
+			)
+		)
+	)
 	(gr_text "1.8V\n"
 		(at 140.25 81.8 0)
@@
 		)
 	)
-	(gr_text "Trigger Output FMC 1.0\nOsprey DCS 2026\n"
+	(gr_text "Trigger Output FMC 1.1\nOsprey DCS 2026\n"
 		(at 186.03 71.845 90)
 		(layer "B.SilkS")
