File: trigger-output-fmc.kicad_sch (KiCad schematic)
At the start: 0 parts

Commit message: Revision based on pre-production
-Added pull-down on the OE for the Digital output buffers
- increase board edge (was 0.3mm, but via and traces are 0.5mm away now)
- move power vias away from board edge
- Increase power via size from 0.6mm/0.3mm to 0.8mm/0.4mm in a couple of places
- Naming of level shifter output enable changed to make function clear throughout the design.
- Revised SMPS layout slightly to better use the space.
Other:
- sheet FMC ports: added Cleaner_LevelShift_~{OE}_0, Cleaner_LevelShift_~{OE}_1; removed Cleaner_~{OE}_0, Cleaner_~{OE}_1
- sheet Level Shifter ports: added Cleaner_LevelShift_~{OE}_0, Cleaner_LevelShift_~{OE}_1; removed OE_Faults_0, OE_Faults_1
Changed lines of the file:
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@@
-			)
-		)
-		(pin "OE_Faults_0" input
-			(at 180.34 86.36 0)
-			(effects
-				(font
-					(size 1.27 1.27)
-				)
-				(justify right)
-			)
-		)
-		(pin "OE_Faults_1" input
-			(at 180.34 99.06 0)
-			(effects
-				(font
-					(size 1.27 1.27)
-				)
-				(justify right)
 			)
 		)
@@
 				)
 				(justify left)
+			)
+		)
+		(pin "Cleaner_LevelShift_~{OE}_0" input
+			(at 180.34 86.36 0)
+			(effects
+				(font
+					(size 1.27 1.27)
+				)
+				(justify right)
+			)
+		)
+		(pin "Cleaner_LevelShift_~{OE}_1" input
+			(at 180.34 99.06 0)
+			(effects
+				(font
+					(size 1.27 1.27)
+				)
+				(justify right)
 			)
 		)
@@
 			)
 		)
-		(pin "Cleaner_~{OE}_0" output
-			(at 208.28 86.36 180)
-			(effects
-				(font
-					(size 1.27 1.27)
-				)
-				(justify left)
-			)
-		)
-		(pin "Cleaner_~{OE}_1" output
-			(at 208.28 99.06 180)
-			(effects
-				(font
-					(size 1.27 1.27)
-				)
-				(justify left)
-			)
-		)
 		(pin "{Digital_LVDS}" output
 			(at 208.28 44.45 180)
@@
 			(effects
 				(font
+					(size 1.27 1.27)
+				)
+				(justify left)
+			)
+		)
+		(pin "Cleaner_LevelShift_~{OE}_0" output
+			(at 208.28 86.36 180)
+			(effects
+				(font
+					(size 1.27 1.27)
+				)
+				(justify left)
+			)
+		)
+		(pin "Cleaner_LevelShift_~{OE}_1" output
+			(at 208.28 99.06 180)
+			(effects
+				(font
